File: new_student.kicad_pcb (KiCad board)
At the start: 2 copper layers, 70.8 x 69 mm, 39 parts, among them IC1 NCV7351D1ER2G, IC2 TA78L05F_F_, IC3 TA78L05F_F_, J1 RJ45_LED_Shielded, J10 Conn_01x04_Pin, J11 Conn_01x04_Pin, J12 Conn_01x04_Pin, J13 Conn_01x02_Pin, J14 Conn_01x02_Pin, J15 Conn_01x02_Pin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

Commit message: Add files via upload
Parts:
- J9: footprint Connector_PinHeader_2.54mm:PinHeader_1x04_P2.54mm_Vertical -> Library:encoder_connect
- moved J9 9.42 mm to (61.8, 118.2), turned to 180 degrees
- moved C2 5.35 mm to (97.7, 68.0)
- moved J5 5.00 mm to (78.9, 117.7), turned to 180 degrees
- moved J4 5.00 mm to (75.2, 117.7), turned to 180 degrees
- moved J3 4.95 mm to (71.5, 117.7), turned to 180 degrees
Connections:
- J13 pad 2: 3v3 -> 5V
- J3 pad 2: servo0 -> VCC
- J3 pad 3: VCC -> servo0
- J4 pad 2: servo1 -> VCC
- J4 pad 3: VCC -> servo1
- J5 pad 2: servo2 -> VCC
- J5 pad 3: VCC -> servo2
Routing:
- net /CAN_ENA: track 7.65 -> 64.8 mm, vias 0 -> 2
- net VCC: track 41.5 -> 0.00 mm
- net 3v3: track 46.0 -> 12.6 mm
- net /ENC_B: track 17.8 -> 33.0 mm
- net GND: track 38.5 -> 28.2 mm
- net /ENC_A: track 18.5 -> 14.4 mm
- net servo2: track 9.63 -> 6.00 mm
- net servo0: track 9.16 -> 6.49 mm
- net servo1: track 9.13 -> 6.89 mm
- net 5V: track 2.10 -> 0.00 mm
- removed copper zone on F.Cu, net /CAN_ENA
