File: new_student.kicad_sch (KiCad schematic)
At the start: 39 parts, among them IC1 NCV7351D1ER2G, IC2 TA78L05F_F_, IC3 TA78L05F_F_, J1 RJ45_LED_Shielded, J10 Conn_01x04_Pin, J11 Conn_01x04_Pin, J12 Conn_01x04_Pin, J13 Conn_01x02_Pin, J14 Conn_01x02_Pin, J15 Conn_01x02_Pin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

Commit message: Add files via upload
いろいろ変えた
Parts:
- removed J13: Conn_01x02_Pin, Connector_PinHeader_2.54mm:PinHeader_1x02_P2.54mm_Vertical, symbol Connector:Conn_01x02_Pin
- added H1, H2: MountingHole, MountingHole:MountingHole_3.2mm_M3, symbol Mechanical:MountingHole
- J9: footprint Connector_PinHeader_2.54mm:PinHeader_1x04_P2.54mm_Vertical -> Library:encoder_connect
Connections:
- net VCC: now also J3.2 (Pin_2), J4.2 (Pin_2), J5.2 (Pin_2); no longer J3.3 (Pin_3), J4.3 (Pin_3), J5.3 (Pin_3)
- net servo0: now also J3.3 (Pin_3); no longer J3.2 (Pin_2)
- net servo1: now also J4.3 (Pin_3); no longer J4.2 (Pin_2)
- net servo2: now also J5.3 (Pin_3); no longer J5.2 (Pin_2)
Changed lines of the file:
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@@
-    (stroke (width 0) (type default))
-  )
-  (wire (pts (xy 382.27 285.75) (xy 378.46 285.75))
     (stroke (width 0) (type default))
   )
@@
   )
   (wire (pts (xy 476.25 232.41) (xy 490.22 232.41))
-    (stroke (width 0) (type default))
-  )
-  (wire (pts (xy 382.27 283.21) (xy 378.46 283.21))
     (stroke (width 0) (type default))
   )
@@
     )
   )
-  (global_label "EMS_button" (shape bidirectional) (at 382.27 283.21 0) (fields_autoplaced)
-    (effects (font (size 1.27 1.27)) (justify left))
-    (property "Intersheetrefs" "${INTERSHEET_REFS}" (at 397.1914 283.21 0)
-      (effects (font (size 1.27 1.27)) (justify left) hide)
-    )
-  )
   (global_label "5V" (shape bidirectional) (at 434.34 217.17 180) (fields_autoplaced)
     (effects (font (size 1.27 1.27)) (justify right))
@@
     )
   )
-  (global_label "VCC" (shape bidirectional) (at 337.82 309.88 0) (fields_autoplaced)
-    (effects (font (size 1.27 1.27)) (justify left))
-    (property "Intersheetrefs" "${INTERSHEET_REFS}" (at 345.5451 309.88 0)
+  (global_label "VCC" (shape bidirectional) (at 337.82 307.34 0) (fields_autoplaced)
+    (effects (font (size 1.27 1.27)) (justify left))
+    (property "Intersheetrefs" "${INTERSHEET_REFS}" (at 345.5451 307.34 0)
       (effects (font (size 1.27 1.27)) (justify left) hide)
     )
@@
     )
   )
-  (global_label "servo0" (shape bidirectional) (at 317.5 307.34 0) (fields_autoplaced)
-    (effects (font (size 1.27 1.27)) (justify left))
-    (property "Intersheetrefs" "${INTERSHEET_REFS}" (at 327.8255 307.34 0)
+  (global_label "servo0" (shape bidirectional) (at 317.5 309.88 0) (fields_autoplaced)
+    (effects (font (size 1.27 1.27)) (justify left))
+    (property "Intersheetrefs" "${INTERSHEET_REFS}" (at 327.8255 309.88 0)
       (effects (font (size 1.27 1.27)) (justify left) hide)
     )
@@
     )
   )
-  (global_label "servo1" (shape bidirectional) (at 337.82 307.34 0) (fields_autoplaced)
-    (effects (font (size 1.27 1.27)) (justify left))
-    (property "Intersheetrefs" "${INTERSHEET_REFS}" (at 348.1455 307.34 0)
+  (global_label "servo1" (shape bidirectional) (at 337.82 309.88 0) (fields_autoplaced)
+    (effects (font (size 1.27 1.27)) (justify left))
+    (property "Intersheetrefs" "${INTERSHEET_REFS}" (at 348.1455 309.88 0)
       (effects (font (size 1.27 1.27)) (justify left) hide)
     )
@@
     )
   )
-  (global_label "servo2" (shape bidirectional) (at 356.87 307.34 0) (fields_autoplaced)
-    (effects (font (size 1.27 1.27)) (justify left))
-    (property "Intersheetrefs" "${INTERSHEET_REFS}" (at 367.1955 307.34 0)
+  (global_label "servo2" (shape bidirectional) (at 356.87 309.88 0) (fields_autoplaced)
+    (effects (font (size 1.27 1.27)) (justify left))
+    (property "Intersheetrefs" "${INTERSHEET_REFS}" (at 367.1955 309.88 0)
       (effects (font (size 1.27 1.27)) (justify left) hide)
     )
@@
     )
   )
-  (global_label "VCC" (shape bidirectional) (at 317.5 309.88 0) (fields_autoplaced)
-    (effects (font (size 1.27 1.27)) (justify left))
-    (property "Intersheetrefs" "${INTERSHEET_REFS}" (at 325.2251 309.88 0)
+  (global_label "VCC" (shape bidirectional) (at 317.5 307.34 0) (fields_autoplaced)
+    (effects (font (size 1.27 1.27)) (justify left))
+    (property "Intersheetrefs" "${INTERSHEET_REFS}" (at 325.2251 307.34 0)
       (effects (font (size 1.27 1.27)) (justify left) hide)
     )
@@
     )
   )
-  (global_label "VCC" (shape bidirectional) (at 356.87 309.88 0) (fields_autoplaced)
-    (effects (font (size 1.27 1.27)) (justify left))
-    (property "Intersheetrefs" "${INTERSHEET_REFS}" (at 364.5951 309.88 0)
+  (global_label "VCC" (shape bidirectional) (at 356.87 307.34 0) (fields_autoplaced)
+    (effects (font (size 1.27 1.27)) (justify left))
+    (property "Intersheetrefs" "${INTERSHEET_REFS}" (at 364.5951 307.34 0)
       (effects (font (size 1.27 1.27)) (justify left) hide)
     )
@@
     (effects (font (size 1.27 1.27)) (justify left))
     (property "Intersheetrefs" "${INTERSHEET_REFS}" (at 330.0631 242.57 0)
-      (effects (font (size 1.27 1.27)) (justify left) hide)
-    )
-  )
-  (global_label "3v3" (shape bidirectional) (at 382.27 285.75 0) (fields_autoplaced)
-    (effects (font (size 1.27 1.27)) (justify left))
-    (property "Intersheetrefs" "${INTERSHEET_REFS}" (at 389.7531 285.75 0)
       (effects (font (size 1.27 1.27)) (justify left) hide)
     )
@@
       (effects (font (size 1.27 1.27)))
     )
-    (property "Footprint" "Connector_PinHeader_2.54mm:PinHeader_1x04_P2.54mm_Vertical" (at 232.41 236.22 0)
+    (property "Footprint" "Library:encoder_connect" (at 232.41 236.22 0)
       (effects (font (size 1.27 1.27)) hide)
     )
@@
         (path "/db0bf1f5-8558-40f6-a79d-8bb07620be8f"
           (reference "J18") (unit 1)
+        )
+      )
+    )
+  )
+  (symbol (lib_id "Mechanical:MountingHole") (at 473.71 314.96 0) (unit 1)
+    (in_bom yes) (on_board yes) (dnp no) (fields_autoplaced)
+    (property "Reference" "H2" (at 476.25 313.69 0)
+      (effects (font (size 1.27 1.27)) (justify left))
+    )
+    (property "Value" "MountingHole" (at 476.25 316.23 0)
+      (effects (font (size 1.27 1.27)) (justify left))
+    )
+    (property "Footprint" "MountingHole:MountingHole_3.2mm_M3" (at 473.71 314.96 0)
+      (effects (font (size 1.27 1.27)) hide)
+    )
+    (property "Datasheet" "~" (at 473.71 314.96 0)
+      (effects (font (size 1.27 1.27)) hide)
+    )
+    (instances
+      (project "new_student"
+        (path "/db0bf1f5-8558-40f6-a79d-8bb07620be8f"
+          (reference "H2") (unit 1)
         )
       )
@@
     )
   )
+  (symbol (lib_id "Mechanical:MountingHole") (at 455.93 314.96 0) (unit 1)
+    (in_bom yes) (on_board yes) (dnp no) (fields_autoplaced)
+    (property "Reference" "H1" (at 458.47 313.69 0)
+      (effects (font (size 1.27 1.27)) (justify left))
+    )
+    (property "Value" "MountingHole" (at 458.47 316.23 0)
+      (effects (font (size 1.27 1.27)) (justify left))
+    )
+    (property "Footprint" "MountingHole:MountingHole_3.2mm_M3" (at 455.93 314.96 0)
+      (effects (font (size 1.27 1.27)) hide)
+    )
+    (property "Datasheet" "~" (at 455.93 314.96 0)
+      (effects (font (size 1.27 1.27)) hide)
+    )
+    (instances
+      (project "new_student"
+        (path "/db0bf1f5-8558-40f6-a79d-8bb07620be8f"
+          (reference "H1") (unit 1)
+        )
+      )
+    )
+  )
   (symbol (lib_id "Connector:Conn_01x03_Pin") (at 331.47 307.34 0) (unit 1)
     (in_bom yes) (on_board yes) (dnp no) (fields_autoplaced)
@@
         )
       )
-    )
-  )
-  (symbol (lib_id "Connector:Conn_01x02_Pin") (at 373.38 283.21 0) (unit 1)
-    (in_bom yes) (on_board yes) (dnp no) (fields_autoplaced)
-    (property "Reference" "J13" (at 374.015 278.13 0)
-      (effects (font (size 1.27 1.27)))
-    )
-    (property "Value" "Conn_01x02_Pin" (at 374.015 280.67 0)
-      (effects (font (size 1.27 1.27)))
-    )
-    (property "Footprint" "Connector_PinHeader_2.54mm:PinHeader_1x02_P2.54mm_Vertical" (at 373.38 283.21 0)
-      (effects (font (size 1.27 1.27)) hide)
-    )
-    (property "Datasheet" "~" (at 373.38 283.21 0)
-      (effects (font (size 1.27 1.27)) hide)
-    )
-    (pin "1")
-    (pin "2")
-    (instances
-      (project "new_student"
-        (path "/db0bf1f5-8558-40f6-a79d-8bb07620be8f"
-          (reference "J13") (unit 1)
-        )
-      )
